File: radio.kicad_sch (KiCad schematic)
At the start: 21 parts, among them IC12 TPS22975, IC6 SN74LVC244A, U2 E22-900M30S

Commit message: name change to Loriques
Parts:
- C29, C34, C40, C48, C50, C61, C63, C72, C73: symbol autonode:CAP0402 -> Loriques:CAP0402
- C47: symbol autonode:CAP1206 -> Loriques:CAP1206
- C62, C64: symbol autonode:CAP1210 -> Loriques:CAP1210
- FL2: footprint autonode:YFF31HC2A104MT000N -> Loriques:YFF31HC2A104MT000N; symbol autonode:YFF31HC2A104MT000N -> Loriques:YFF31HC2A104MT000N
- IC12: footprint autonode:WSON8 -> Loriques:WSON8; symbol autonode:TPS22975 -> Loriques:TPS22975
- IC6: footprint autonode:R-PVQFN-N20 -> Loriques:R-PVQFN-N20; symbol autonode:SN74LVC244A -> Loriques:SN74LVC244A
- R32, R33: symbol autonode:RESISTOR0402-RES -> Loriques:RESISTOR0402-RES
- S_3V3, TP6, TP8: footprint autonode:PAD.03X.05 -> TestPoint:TestPoint_Pad_D1.5mm; symbol autonode:TEST-POINT3X5 -> Connector:TestPoint
- U2: footprint autonode:E22-900M30S -> Loriques:E22-900M30S; symbol autonode:E22-900M30S -> Loriques:E22-900M30S
Connections:
- net 3V3: now also TP6.1; no longer TP6.0 (1)
- net RADIO_3V3: now also S_3V3.1; no longer S_3V3.0 (1)
- net RADIO_EN: now also TP8.1; no longer TP8.0 (1)
Changed lines of the file:
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@@
 	)
 	(symbol
-		(lib_id "autonode:TEST-POINT3X5")
+		(lib_id "Connector:TestPoint")
 		(at 91.44 73.66 270)
 		(unit 1)
@@
 			)
 		)
-		(property "Footprint" "autonode:PAD.03X.05"
+		(property "Footprint" "TestPoint:TestPoint_Pad_D1.5mm"
+			(at 91.44 78.74 0)
+			(effects
+				(font
+					(size 1.27 1.27)
+				)
+				(hide yes)
+			)
+		)
+		(property "Datasheet" "~"
+			(at 91.44 78.74 0)
+			(effects
+				(font
+					(size 1.27 1.27)
+				)
+				(hide yes)
+			)
+		)
+		(property "Description" "test point"
 			(at 91.44 73.66 0)
 			(effects
@@
 			)
 		)
-		(property "Datasheet" ""
-			(at 91.44 73.66 0)
-			(effects
-				(font
-					(size 1.27 1.27)
-				)
-				(hide yes)
-			)
-		)
-		(property "Description" "Bare copper test points for troubleshooting or ICT"
-			(at 91.44 73.66 0)
-			(effects
-				(font
-					(size 1.27 1.27)
-				)
-				(hide yes)
-			)
-		)
-		(pin "0"
-		)
-		(instances
-			(project "AutoNode"
+		(pin "1"
+		)
+		(instances
+			(project "Loriques"
 				(path "/23714a9e-6212-41ed-9d80-e983f828d45f/31a08346-8aff-492d-a666-d252f0663a7c"
 					(reference "TP8")
@@
 	)
 	(symbol
-		(lib_id "autonode:RESISTOR0402-RES")
+		(lib_id "Loriques:RESISTOR0402-RES")
 		(at 190.5 60.96 90)
 		(unit 1)
@@
 		)
 		(instances
-			(project "AutoNode"
+			(project "Loriques"
 				(path "/23714a9e-6212-41ed-9d80-e983f828d45f/31a08346-8aff-492d-a666-d252f0663a7c"
 					(reference "R32")
@@
 	)
 	(symbol
-		(lib_id "autonode:E22-900M30S")
+		(lib_id "Loriques:E22-900M30S")
 		(at 119.38 118.11 0)
 		(unit 1)
@@
 			)
 		)
-		(property "Footprint" "autonode:E22-900M30S"
+		(property "Footprint" "Loriques:E22-900M30S"
 			(at 118.11 139.954 0)
 			(effects
@@
 	)
 	(symbol
-		(lib_id "autonode:TEST-POINT3X5")
+		(lib_id "Connector:TestPoint")
 		(at 149.86 63.5 0)
 		(unit 1)
@@
 			)
 		)
-		(property "Footprint" "autonode:PAD.03X.05"
+		(property "Footprint" "TestPoint:TestPoint_Pad_D1.5mm"
+			(at 154.94 63.5 0)
+			(effects
+				(font
+					(size 1.27 1.27)
+				)
+				(hide yes)
+			)
+		)
+		(property "Datasheet" "~"
+			(at 154.94 63.5 0)
+			(effects
+				(font
+					(size 1.27 1.27)
+				)
+				(hide yes)
+			)
+		)
+		(property "Description" "test point"
 			(at 149.86 63.5 0)
 			(effects
@@
 			)
 		)
-		(property "Datasheet" ""
-			(at 149.86 63.5 0)
-			(effects
-				(font
-					(size 1.27 1.27)
-				)
-				(hide yes)
-			)
-		)
-		(property "Description" "Bare copper test points for troubleshooting or ICT"
-			(at 149.86 63.5 0)
-			(effects
-				(font
-					(size 1.27 1.27)
-				)
-				(hide yes)
-			)
-		)
-		(pin "0"
-		)
-		(instances
-			(project "AutoNode"
+		(pin "1"
+		)
+		(instances
+			(project "Loriques"
 				(path "/23714a9e-6212-41ed-9d80-e983f828d45f/31a08346-8aff-492d-a666-d252f0663a7c"
 					(reference "S_3V3")
@@
 	)
 	(symbol
-		(lib_id "autonode:CAP1206")
+		(lib_id "Loriques:CAP1206")
 		(at 73.66 35.56 0)
 		(unit 1)
@@
 		)
 		(instances
-			(project "AutoNode"
+			(project "Loriques"
 				(path "/23714a9e-6212-41ed-9d80-e983f828d45f/31a08346-8aff-492d-a666-d252f0663a7c"
 					(reference "C47")
@@
 	)
 	(symbol
-		(lib_id "autonode:CAP0402")
+		(lib_id "Loriques:CAP0402")
 		(at 121.92 35.56 0)
 		(unit 1)
@@
 		)
 		(instances
-			(project "AutoNode"
+			(project "Loriques"
 				(path "/23714a9e-6212-41ed-9d80-e983f828d45f/31a08346-8aff-492d-a666-d252f0663a7c"
 					(reference "C50")
@@
 	)
 	(symbol
-		(lib_id "autonode:TEST-POINT3X5")
+		(lib_id "Connector:TestPoint")
 		(at 83.82 63.5 90)
 		(unit 1)
@@
 			)
 		)
-		(property "Footprint" "autonode:PAD.03X.05"
+		(property "Footprint" "TestPoint:TestPoint_Pad_D1.5mm"
+			(at 83.82 58.42 0)
+			(effects
+				(font
+					(size 1.27 1.27)
+				)
+				(hide yes)
+			)
+		)
+		(property "Datasheet" "~"
+			(at 83.82 58.42 0)
+			(effects
+				(font
+					(size 1.27 1.27)
+				)
+				(hide yes)
+			)
+		)
+		(property "Description" "test point"
 			(at 83.82 63.5 0)
 			(effects
@@
 			)
 		)
-		(property "Datasheet" ""
-			(at 83.82 63.5 0)
-			(effects
-				(font
-					(size 1.27 1.27)
-				)
-				(hide yes)
-			)
-		)
-		(property "Description" "Bare copper test points for troubleshooting or ICT"
-			(at 83.82 63.5 0)
-			(effects
-				(font
-					(size 1.27 1.27)
-				)
-				(hide yes)
-			)
-		)
-		(pin "0"
-		)
-		(instances
-			(project "AutoNode"
+		(pin "1"
+		)
+		(instances
+			(project "Loriques"
 				(path "/23714a9e-6212-41ed-9d80-e983f828d45f/31a08346-8aff-492d-a666-d252f0663a7c"
 					(reference "TP6")
@@
 	)
 	(symbol
-		(lib_id "autonode:CAP0402")
+		(lib_id "Loriques:CAP0402")
 		(at 91.44 35.56 0)
 		(unit 1)
@@
 		)
 		(instances
-			(project "AutoNode"
+			(project "Loriques"
 				(path "/23714a9e-6212-41ed-9d80-e983f828d45f/31a08346-8aff-492d-a666-d252f0663a7c"
 					(reference "C63")
@@
 	)
 	(symbol
-		(lib_id "autonode:CAP0402")
+		(lib_id "Loriques:CAP0402")
 		(at 106.68 35.56 0)
 		(unit 1)
@@
 		)
 		(instances
-			(project "AutoNode"
+			(project "Loriques"
 				(path "/23714a9e-6212-41ed-9d80-e983f828d45f/31a08346-8aff-492d-a666-d252f0663a7c"
 					(reference "C48")
@@
 	)
 	(symbol
-		(lib_id "autonode:CAP0402")
+		(lib_id "Loriques:CAP0402")
 		(at 25.4 35.56 0)
 		(unit 1)
@@
 		)
 		(instances
-			(project "AutoNode"
+			(project "Loriques"
 				(path "/23714a9e-6212-41ed-9d80-e983f828d45f/31a08346-8aff-492d-a666-d252f0663a7c"
 					(reference "C73")
@@
 	)
 	(symbol
-		(lib_id "autonode:CAP1210")
+		(lib_id "Loriques:CAP1210")
 		(at 157.48 35.56 0)
 		(unit 1)
@@
 		)
 		(instances
-			(project "AutoNode"
+			(project "Loriques"
 				(path "/23714a9e-6212-41ed-9d80-e983f828d45f/31a08346-8aff-492d-a666-d252f0663a7c"
 					(reference "C62")
@@
 	)
 	(symbol
-		(lib_id "autonode:SN74LVC244A")
+		(lib_id "Loriques:SN74LVC244A")
 		(at 223.52 83.82 0)
 		(unit 1)
@@
 			)
 		)
-		(property "Footprint" "autonode:R-PVQFN-N20"
+		(property "Footprint" "Loriques:R-PVQFN-N20"
 			(at 223.52 83.82 0)
 			(effects
@@
 		)
 		(instances
-			(project "AutoNode"
+			(project "Loriques"
 				(path "/23714a9e-6212-41ed-9d80-e983f828d45f/31a08346-8aff-492d-a666-d252f0663a7c"
 					(reference "IC6")
@@
 	)
 	(symbol
-		(lib_id "autonode:CAP0402")
+		(lib_id "Loriques:CAP0402")
 		(at 139.7 35.56 0)
 		(unit 1)
@@
 		)
 		(instances
-			(project "AutoNode"
+			(project "Loriques"
 				(path "/23714a9e-6212-41ed-9d80-e983f828d45f/31a08346-8aff-492d-a666-d252f0663a7c"
 					(reference "C61")
@@
 	)
 	(symbol
-		(lib_id "autonode:RESISTOR0402-RES")
+		(lib_id "Loriques:RESISTOR0402-RES")
 		(at 180.34 60.96 90)
 		(unit 1)
@@
 		)
 		(instances
-			(project "AutoNode"
+			(project "Loriques"
 				(path "/23714a9e-6212-41ed-9d80-e983f828d45f/31a08346-8aff-492d-a666-d252f0663a7c"
 					(reference "R33")
@@
 	)
 	(symbol
-		(lib_id "autonode:CAP0402")
+		(lib_id "Loriques:CAP0402")
 		(at 71.12 71.12 0)
 		(unit 1)
@@
 		)
 		(instances
-			(project "AutoNode"
+			(project "Loriques"
 				(path "/23714a9e-6212-41ed-9d80-e983f828d45f/31a08346-8aff-492d-a666-d252f0663a7c"
 					(reference "C34")
@@
 	)
 	(symbol
-		(lib_id "autonode:CAP0402")
+		(lib_id "Loriques:CAP0402")
 		(at 144.78 76.2 0)
 		(unit 1)
@@
 		)
 		(instances
-			(project "AutoNode"
+			(project "Loriques"
 				(path "/23714a9e-6212-41ed-9d80-e983f828d45f/31a08346-8aff-492d-a666-d252f0663a7c"
 					(reference "C40")
@@
 	)
 	(symbol
-		(lib_id "autonode:TPS22975")
+		(lib_id "Loriques:TPS22975")
 		(at 116.84 68.58 0)
 		(unit 1)
@@
 			)
 		)
-		(property "Footprint" "autonode:WSON8"
+		(property "Footprint" "Loriques:WSON8"
 			(at 116.84 68.58 0)
 			(effects
@@
 		)
 		(instances
-			(project "AutoNode"
+			(project "Loriques"
 				(path "/23714a9e-6212-41ed-9d80-e983f828d45f/31a08346-8aff-492d-a666-d252f0663a7c"
 					(reference "IC12")
@@
 	)
 	(symbol
-		(lib_id "autonode:CAP0402")
+		(lib_id "Loriques:CAP0402")
 		(at 185.42 104.14 0)
 		(unit 1)
@@
 		)
 		(instances
-			(project "AutoNode"
+			(project "Loriques"
 				(path "/23714a9e-6212-41ed-9d80-e983f828d45f/31a08346-8aff-492d-a666-d252f0663a7c"
 					(reference "C29")
@@
 	)
 	(symbol
-		(lib_id "autonode:CAP1210")
+		(lib_id "Loriques:CAP1210")
 		(at 172.72 35.56 0)
 		(unit 1)
@@
 		)
 		(instances
-			(project "AutoNode"
+			(project "Loriques"
 				(path "/23714a9e-6212-41ed-9d80-e983f828d45f/31a08346-8aff-492d-a666-d252f0663a7c"
 					(reference "C64")
@@
 	)
 	(symbol
-		(lib_id "autonode:YFF31HC2A104MT000N")
+		(lib_id "Loriques:YFF31HC2A104MT000N")
 		(at 43.18 27.94 0)
 		(unit 1)
@@
 			)
 		)
-		(property "Footprint" "autonode:YFF31HC2A104MT000N"
+		(property "Footprint" "Loriques:YFF31HC2A104MT000N"
 			(at 43.18 27.94 0)
 			(effects
@@
 		)
 		(instances
-			(project "AutoNode"
+			(project "Loriques"
 				(path "/23714a9e-6212-41ed-9d80-e983f828d45f/31a08346-8aff-492d-a666-d252f0663a7c"
 					(reference "FL2")
@@
 	)
 	(symbol
-		(lib_id "autonode:CAP0402")
+		(lib_id "Loriques:CAP0402")
 		(at 58.42 35.56 0)
 		(unit 1)
@@
 		)
 		(instances
-			(project "AutoNode"
+			(project "Loriques"
 				(path "/23714a9e-6212-41ed-9d80-e983f828d45f/31a08346-8aff-492d-a666-d252f0663a7c"
 					(reference "C72")

Commit message: added logo to schematic sheets
Other:
- title: (none) -> Loriques
- moved on the sheet: C29, C34, C40, C47, C48, C50, C61, C62, C63, C64, C72, C73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

Commit message: more 3D parts. changed out the temp/humidity sensor for an instock one
Connections:
- net BUSY: no longer IC6.P$17 (2IN4), U2.14 (BUSY)
- net MISO: no longer IC6.P$2 (1IN1), U2.16 (MISO)
- net MOSI: no longer IC6.P$16 (1OUT2), U2.17 (MOSI)
- net NSS: no longer IC6.P$12 (1OUT4), U2.19 (NSS)
- net RST: no longer IC6.P$5 (2OUT3), U2.15 (~{RST})
- net RXEN: no longer IC6.P$9 (2OUT1), U2.6 (RXEN)
- net SCK: no longer IC6.P$14 (1OUT3), U2.18 (SCK)
- net TXEN: no longer IC6.P$7 (2OUT2), U2.7 (TXEN)
- new net BUSY_RADIO: IC6.P$17 (2IN4), U2.14 (BUSY)
- new net MISO_RADIO: IC6.P$2 (1IN1), U2.16 (MISO)
- new net MOSI_RADIO: IC6.P$16 (1OUT2), U2.17 (MOSI)
- new net NSS_RADIO: IC6.P$12 (1OUT4), U2.19 (NSS)
- new net RST_RADIO: IC6.P$5 (2OUT3), U2.15 (~{RST})
- new net RXEN_RADIO: IC6.P$9 (2OUT1), U2.6 (RXEN)
- new net SCK_RADIO: IC6.P$14 (1OUT3), U2.18 (SCK)
- new net TXEN_RADIO: IC6.P$7 (2OUT2), U2.7 (TXEN)
Changed lines of the file:
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@@
 	(wire
 		(pts
-			(xy 110.49 124.46) (xy 120.65 124.46)
+			(xy 106.68 124.46) (xy 120.65 124.46)
 		)
 		(stroke
@@
 	(wire
 		(pts
-			(xy 110.49 129.54) (xy 120.65 129.54)
+			(xy 106.68 129.54) (xy 120.65 129.54)
 		)
 		(stroke
@@
 	(wire
 		(pts
-			(xy 110.49 132.08) (xy 120.65 132.08)
+			(xy 106.68 132.08) (xy 120.65 132.08)
 		)
 		(stroke
@@
 	(wire
 		(pts
-			(xy 110.49 142.24) (xy 120.65 142.24)
+			(xy 106.68 142.24) (xy 120.65 142.24)
 		)
 		(stroke
@@
 	(wire
 		(pts
-			(xy 110.49 144.78) (xy 120.65 144.78)
+			(xy 106.68 144.78) (xy 120.65 144.78)
 		)
 		(stroke
@@
 	(wire
 		(pts
-			(xy 110.49 134.62) (xy 120.65 134.62)
+			(xy 106.68 134.62) (xy 120.65 134.62)
 		)
 		(stroke
@@
 	(wire
 		(pts
-			(xy 146.05 147.32) (xy 156.21 147.32)
+			(xy 146.05 147.32) (xy 161.29 147.32)
 		)
 		(stroke
@@
 	(wire
 		(pts
-			(xy 110.49 137.16) (xy 120.65 137.16)
+			(xy 106.68 137.16) (xy 120.65 137.16)
 		)
 		(stroke
@@
 	(wire
 		(pts
-			(xy 156.21 132.08) (xy 146.05 132.08)
+			(xy 161.29 132.08) (xy 146.05 132.08)
 		)
 		(stroke
@@
 		)
 	)
-	(label "BUSY"
+	(label "BUSY_RADIO"
 		(at 214.63 113.03 0)
 		(effects
@@
 		)
 	)
-	(label "NSS"
+	(label "NSS_RADIO"
 		(at 265.43 97.79 180)
 		(effects
@@
 		)
 	)
-	(label "MISO"
+	(label "MISO_RADIO"
 		(at 214.63 90.17 0)
 		(effects
@@
 		)
 	)
-	(label "NSS"
-		(at 110.49 137.16 0)
+	(label "NSS_RADIO"
+		(at 106.68 137.16 0)
 		(effects
 			(font
@@
 		)
 	)
-	(label "SCK"
-		(at 110.49 134.62 0)
-		(effects
-			(font
-				(size 1.27 1.27)
-			)
-			(justify left bottom)
-		)
-	)
-	(label "RXEN"
-		(at 110.49 142.24 0)
+	(label "SCK_RADIO"
+		(at 106.68 134.62 0)
+		(effects
+			(font
+				(size 1.27 1.27)
+			)
+			(justify left bottom)
+		)
+	)
+	(label "RXEN_RADIO"
+		(at 106.68 142.24 0)
 		(effects
 			(font
@@
 		)
 	)
-	(label "MOSI"
+	(label "MOSI_RADIO"
 		(at 265.43 92.71 180)
 		(effects
@@
 	)
 	(label "GND"
-		(at 156.21 147.32 180)
+		(at 161.29 147.32 180)
 		(effects
 			(font
@@
 		)
 	)
-	(label "RXEN"
+	(label "RXEN_RADIO"
 		(at 265.43 105.41 180)
 		(effects
@@
 		)
 	)
-	(label "TXEN"
+	(label "TXEN_RADIO"
 		(at 265.43 107.95 180)
 		(effects
@@
 		)
 	)
-	(label "RST"
+	(label "RST_RADIO"
 		(at 265.43 110.49 180)
 		(effects
@@
 		)
 	)
-	(label "BUSY"
-		(at 156.21 132.08 180)
+	(label "BUSY_RADIO"
+		(at 161.29 132.08 180)
 		(effects
 			(font
@@
 		)
 	)
-	(label "MOSI"
-		(at 110.49 129.54 0)
+	(label "MOSI_RADIO"
+		(at 106.68 129.54 0)
 		(effects
 			(font
@@
 		)
 	)
-	(label "TXEN"
-		(at 110.49 144.78 0)
+	(label "TXEN_RADIO"
+		(at 106.68 144.78 0)
 		(effects
 			(font
@@
 		)
 	)
-	(label "MISO"
-		(at 110.49 132.08 0)
-		(effects
-			(font
-				(size 1.27 1.27)
-			)
-			(justify left bottom)
-		)
-	)
-	(label "SCK"
+	(label "MISO_RADIO"
+		(at 106.68 132.08 0)
+		(effects
+			(font
+				(size 1.27 1.27)
+			)
+			(justify left bottom)
+		)
+	)
+	(label "SCK_RADIO"
 		(at 265.43 95.25 180)
 		(effects
@@
 		)
 	)
-	(label "RST"
-		(at 110.49 124.46 0)
-		(effects
-			(font
+	(label "RST_RADIO"
+		(at 106.68 124.46 0)
+		(effects
+			(font

Commit message: lots of routing, tweaking placement. adding courtyards
Parts:
- IC12: DK (none) -> 296-47228-1-ND; PARTNO (none) -> TPS22975DSGR
Connections:
- net 3V3: now also IC6.20 (VCC); no longer IC6.P$20 (VCC)
- net BUSY: now also IC6.3 (2OUT4); no longer IC6.P$3 (2OUT4)
- net BUSY_RADIO: now also IC6.17 (2IN4); no longer IC6.P$17 (2IN4)
- net GND: now also IC6.10 (GND), IC6.21 (GND); no longer IC6.P$10 (GND), IC6.P$21 (GND), IC6.P$22 (GND), IC6.P$23 (GND), IC6.P$24 (GND), IC6.P$25 (GND), IC6.P$26 (GND), IC6.P$27 (GND)
- net MISO: now also IC6.18 (1OUT1); no longer IC6.P$18 (1OUT1)
- net MISO_RADIO: now also IC6.2 (1IN1); no longer IC6.P$2 (1IN1)
- net MOSI: now also IC6.4 (1IN2); no longer IC6.P$4 (1IN2)
- net MOSI_RADIO: now also IC6.16 (1OUT2); no longer IC6.P$16 (1OUT2)
- net NSS: now also IC6.8 (1IN4); no longer IC6.P$8 (1IN4)
- net NSS_RADIO: now also IC6.12 (1OUT4); no longer IC6.P$12 (1OUT4)
- net RST: now also IC6.15 (2IN3); no longer IC6.P$15 (2IN3)
- net RST_RADIO: now also IC6.5 (2OUT3); no longer IC6.P$5 (2OUT3)
- net RXEN: now also IC6.11 (2IN1); no longer IC6.P$11 (2IN1)
- net RXEN_RADIO: now also IC6.9 (2OUT1); no longer IC6.P$9 (2OUT1)
- net SCK: now also IC6.6 (1IN3); no longer IC6.P$6 (1IN3)
- net SCK_RADIO: now also IC6.14 (1OUT3); no longer IC6.P$14 (1OUT3)
- net TXEN: now also IC6.13 (2IN2); no longer IC6.P$13 (2IN2)
- net TXEN_RADIO: now also IC6.7 (2OUT2); no longer IC6.P$7 (2OUT2)
- net at R32.1: now also IC6.1 (1OE); no longer IC6.P$1 (1OE)
- net at R33.1: now also IC6.19 (2OE); no longer IC6.P$19 (2OE)
Changed lines of the file:
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@@
 			)
 		)
-		(pin "P$1"
-		)
-		(pin "P$10"
-		)
-		(pin "P$11"
-		)
-		(pin "P$12"
-		)
-		(pin "P$13"
-		)
-		(pin "P$14"
-		)
-		(pin "P$15"
-		)
-		(pin "P$16"
-		)
-		(pin "P$17"
-		)
-		(pin "P$18"
-		)
-		(pin "P$19"
-		)
-		(pin "P$2"
-		)
-		(pin "P$20"
-		)
-		(pin "P$21"
-		)
-		(pin "P$22"
-		)
-		(pin "P$23"
-		)
-		(pin "P$24"
-		)
-		(pin "P$25"
-		)
-		(pin "P$26"
-		)
-		(pin "P$27"
-		)
-		(pin "P$3"
-		)
-		(pin "P$4"
-		)
-		(pin "P$5"
-		)
-		(pin "P$6"
-		)
-		(pin "P$7"
-		)
-		(pin "P$8"
-		)
-		(pin "P$9"
+		(pin "5"
+		)
+		(pin "21"
+		)
+		(pin "18"
+		)
+		(pin "20"
+		)
+		(pin "10"
+		)
+		(pin "16"
+		)
+		(pin "14"
+		)
+		(pin "12"
+		)
+		(pin "3"
+		)
+		(pin "9"
+		)
+		(pin "7"
+		)
+		(pin "1"
+		)
+		(pin "2"
+		)
+		(pin "4"
+		)
+		(pin "6"
+		)
+		(pin "8"
+		)
+		(pin "19"
+		)
+		(pin "11"
+		)
+		(pin "13"
+		)
+		(pin "15"
+		)
+		(pin "17"
 		)
 		(instances
@@
 			)
 		)
-		(property "Datasheet" ""
+		(property "Datasheet" "https://www.ti.com/lit/ds/symlink/tps22975.pdf"
 			(at 130.81 85.09 0)
 			(effects
@@
 			)
 		)
-		(property "Description" "TPS22975\nLOAD SWITCH N-CH 6A 8WSON"
+		(property "Description" "LOAD SWITCH N-CH 6A 8WSON"
 			(at 130.81 85.09 0)
 			(effects
 				(font
+					(size 1.27 1.27)
+				)
+				(hide yes)
+			)
+		)
+		(property "PARTNO" "TPS22975DSGR"
+			(at 130.81 98.298 0)
+			(effects
+				(font
+					(size 1.27 1.27)
+				)
+				(hide yes)
+			)
+		)
+		(property "DK" "296-47228-1-ND"
+			(at 130.81 98.298 0)
+			(effects
+				(font
